File: hardware/OmniProbe/OmniProbe.kicad_pcb (KiCad board)
At the start: 2 copper layers, 52.7 x 29.1 mm, 62 parts, among them J1 USB_C_Receptacle_USB2.0_16P, J10 Conn_01x04_Socket, J2 Conn_ARM_JTAG_SWD_10, J6 Conn_01x03_Socket, J7 Conn_01x03_Socket, J8 Conn_01x16_Socket, J9 Conn_01x04_Socket, U1 RP2040, U2 W25Q128JVP, U3 AP2112K-3.3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

Commit message: v0
Parts:
- moved J9 49.5 mm to (146.2, 87.7)
- moved J7 39.4 mm to (162.4, 87.7)
- moved J6 37.7 mm to (166.0, 87.7)
- moved J10 4.39 mm to (115.3, 66.8)
- moved C1 3.97 mm to (132.3, 88.3)
- moved C18 3.97 mm to (141.3, 88.4)
- moved C2 3.97 mm to (133.8, 88.3)
- moved C21 3.97 mm to (142.7, 88.4)
- moved C3 3.97 mm to (135.2, 88.3)
- moved C4 3.97 mm to (130.8, 88.3)
- moved R3 3.97 mm to (138.6, 90.5)
- moved U3 3.97 mm to (138.4, 88.3)
- moved D3 3.85 mm to (128.9, 89.1)
Routing:
- net VBUS: track 8.39 -> 0.00 mm
- net 3V3: track 3.18 -> 0.00 mm
- net Net-(D3-A): track 1.93 -> 0.00 mm
- net Net-(F1-Pad2): track 1.33 -> 0.00 mm
Changed lines of the file:
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@@
 	(footprint "Resistor_SMD:R_0603_1608Metric"
 		(layer "F.Cu")
-		(at 142.583372 90.537086 180)
+		(at 138.617245 90.480817 180)
 		(descr "Resistor SMD 0603 (1608 Metric), square (rectangular) end terminal, IPC-7351 nominal, (Body size source: IPC-SM-782 page 72, https://www.pcb-3d.com/wordpress/wp-content/uploads/ipc-sm-782a_amendment_1_and_2.pdf)")
 		(tags "resistor")
@@
 	(footprint "Capacitor_SMD:C_0603_1608Metric"
 		(layer "F.Cu")
-		(at 145.219904 88.445353 -90)
+		(at 141.253777 88.389084 -90)
 		(descr "Capacitor SMD 0603 (1608 Metric), square (rectangular) end terminal, IPC-7351 nominal, (Body size source: IPC-SM-782 page 76, https://www.pcb-3d.com/wordpress/wp-content/uploads/ipc-sm-782a_amendment_1_and_2.pdf)")
 		(tags "capacitor")
@@
 	(footprint "Connector_PinHeader_2.54mm:PinHeader_1x03_P2.54mm_Vertical"
 		(layer "F.Cu")
-		(at 133.46 68.5 90)
+		(at 165.964168 87.676058 90)
 		(descr "Through hole straight pin header, 1x03, 2.54mm pitch, single row")
 		(tags "Through hole pin header THT 1x03 2.54mm single row")
@@
 	(footprint "Capacitor_SMD:C_0603_1608Metric"
 		(layer "F.Cu")
-		(at 146.691834 88.445353 -90)
+		(at 142.725707 88.389084 -90)
 		(descr "Capacitor SMD 0603 (1608 Metric), square (rectangular) end terminal, IPC-7351 nominal, (Body size source: IPC-SM-782 page 76, https://www.pcb-3d.com/wordpress/wp-content/uploads/ipc-sm-782a_amendment_1_and_2.pdf)")
 		(tags "capacitor")
@@
 	(footprint "Capacitor_SMD:C_0603_1608Metric"
 		(layer "F.Cu")
-		(at 139.199362 88.397967 -90)
+		(at 135.233235 88.341698 -90)
 		(descr "Capacitor SMD 0603 (1608 Metric), square (rectangular) end terminal, IPC-7351 nominal, (Body size source: IPC-SM-782 page 76, https://www.pcb-3d.com/wordpress/wp-content/uploads/ipc-sm-782a_amendment_1_and_2.pdf)")
 		(tags "capacitor")
@@
 	(footprint "Connector_PinHeader_2.54mm:PinHeader_1x03_P2.54mm_Vertical"
 		(layer "F.Cu")
-		(at 127.731383 69 -90)
+		(at 162.411788 87.676058 -90)
 		(descr "Through hole straight pin header, 1x03, 2.54mm pitch, single row")
 		(tags "Through hole pin header THT 1x03 2.54mm single row")
@@
 	(footprint "Capacitor_SMD:C_0603_1608Metric"
 		(layer "F.Cu")
-		(at 134.752996 88.398799 -90)
+		(at 130.786869 88.34253 -90)
 		(descr "Capacitor SMD 0603 (1608 Metric), square (rectangular) end terminal, IPC-7351 nominal, (Body size source: IPC-SM-782 page 76, https://www.pcb-3d.com/wordpress/wp-content/uploads/ipc-sm-782a_amendment_1_and_2.pdf)")
 		(tags "capacitor")
@@
 	(footprint "Capacitor_SMD:C_0603_1608Metric"
 		(layer "F.Cu")
-		(at 136.257634 88.398799 -90)
+		(at 132.291507 88.34253 -90)
 		(descr "Capacitor SMD 0603 (1608 Metric), square (rectangular) end terminal, IPC-7351 nominal, (Body size source: IPC-SM-782 page 76, https://www.pcb-3d.com/wordpress/wp-content/uploads/ipc-sm-782a_amendment_1_and_2.pdf)")
 		(tags "capacitor")
@@
 	(footprint "PCM_SparkFun-Semiconductor-Standard:SOT23-5"
 		(layer "F.Cu")
-		(at 142.317556 88.364506)
+		(at 138.351429 88.308237)
 		(tags "SparkFun")
 		(property "Reference" "U3"
@@
 	(footprint "Capacitor_SMD:C_0603_1608Metric"
 		(layer "F.Cu")
-		(at 137.731716 88.397868 -90)
+		(at 133.765589 88.341599 -90)
 		(descr "Capacitor SMD 0603 (1608 Metric), square (rectangular) end terminal, IPC-7351 nominal, (Body size source: IPC-SM-782 page 76, https://www.pcb-3d.com/wordpress/wp-content/uploads/ipc-sm-782a_amendment_1_and_2.pdf)")
 		(tags "capacitor")
@@
 	(footprint "Connector_PinHeader_2.54mm:PinHeader_1x04_P2.54mm_Vertical"
 		(layer "F.Cu")
-		(at 119.08 69 -90)
+		(at 115.31 66.75 -90)
 		(descr "Through hole straight pin header, 1x04, 2.54mm pitch, single row")
 		(tags "Through hole pin header THT 1x04 2.54mm single row")
@@
 	(footprint "Diode_SMD:D_SOD-123F"
 		(layer "F.Cu")
-		(at 132.747867 89.113136 -90)
+		(at 128.894458 89.056403 -90)
 		(descr "D_SOD-123F")
 		(tags "D_SOD-123F")
@@
 	(footprint "Connector_PinHeader_2.54mm:PinHeader_1x04_P2.54mm_Vertical"
 		(layer "F.Cu")
-		(at 100.274856 68.99389 90)
+		(at 146.158556 87.669053 90)
 		(descr "Through hole straight pin header, 1x04, 2.54mm pitch, single row")
 		(tags "Through hole pin header THT 1x04 2.54mm single row")
@@
 	)
 	(segment
-		(start 130.867812 93.460161)
-		(end 130.867812 92.172055)
-		(width 0.5)
-		(layer "F.Cu")
-		(net "Net-(F1-Pad2)")
-	)
-	(segment
-		(start 130.867812 92.172055)
-		(end 130.837463 92.141706)
-		(width 0.5)
-		(layer "F.Cu")
-		(net "Net-(F1-Pad2)")
-	)
-	(segment
-		(start 130.837463 90.566706)
-		(end 132.694297 90.566706)
-		(width 0.5)
-		(layer "F.Cu")
-		(net "Net-(D3-A)")
-	)
-	(segment
-		(start 132.694297 90.566706)
-		(end 132.747867 90.513136)
-		(width 0.5)
-		(layer "F.Cu")
-		(net "Net-(D3-A)")
-	)
-	(segment
-		(start 144.964057 87.414506)
-		(end 145.219904 87.670353)
-		(width 0.5)
-		(layer "F.Cu")
-		(net "3V3")
-	)
-	(segment
-		(start 143.617656 87.414506)
-		(end 144.964057 87.414506)
-		(width 0.5)
-		(layer "F.Cu")
-		(net "3V3")
-	)
-	(segment
-		(start 145.219904 87.670353)
-		(end 146.691834 87.670353)
-		(width 0.5)
-		(layer "F.Cu")
-		(net "3V3")
-	)
-	(segment
-		(start 139.199263 87.622868)
-		(end 139.199362 87.622967)
-		(width 0.5)
-		(layer "F.Cu")
-		(net "VBUS")
-	)
-	(segment
-		(start 132.747867 87.713136)
-		(end 134.663659 87.713136)
-		(width 0.5)
-		(layer "F.Cu")
-		(net "VBUS")
-	)
-	(segment
-		(start 136.257634 87.623799)
-		(end 137.730785 87.623799)
-		(width 0.5)
-		(layer "F.Cu")
-		(net "VBUS")
-	)
-	(segment
-		(start 134.663659 87.713136)
-		(end 134.752996 87.623799)
-		(width 0.5)
-		(layer "F.Cu")
-		(net "VBUS")
-	)
-	(segment
-		(start 137.731716 87.622868)
-		(end 139.199263 87.622868)
-		(width 0.5)
-		(layer "F.Cu")
-		(net "VBUS")
-	)
-	(segment
-		(start 139.407823 87.414506)
-		(end 139.199362 87.622967)
-		(width 0.5)
-		(layer "F.Cu")
-		(net "VBUS")
-	)
-	(segment
-		(start 141.017456 87.414506)
-		(end 139.407823 87.414506)
-		(width 0.5)
-		(layer "F.Cu")
-		(net "VBUS")
-	)
-	(segment
-		(start 134.752996 87.623799)
-		(end 136.257634 87.623799)
-		(width 0.5)
-		(layer "F.Cu")
-		(net "VBUS")
-	)
-	(segment
-		(start 137.730785 87.623799)
-		(end 137.731716 87.622868)
-		(width 0.5)
-		(layer "F.Cu")
-		(net "VBUS")
-	)
-	(segment

Commit message: V0
Parts:
- removed J8: Conn_01x16_Socket, Connector_PinHeader_2.54mm:PinHeader_1x16_P2.54mm_Vertical
- added J3: Conn_01x20_Socket, Connector_PinHeader_2.54mm:PinHeader_1x20_P2.54mm_Vertical, F.Cu at (122.4, 113.2)
- added J4: Conn_01x06_Socket, Connector_PinHeader_2.54mm:PinHeader_1x06_P2.54mm_Vertical, F.Cu at (157.9, 87.7)
- added R21: 47R, Resistor_SMD:R_0603_1608Metric, F.Cu at (124.7, 60.0)
- added R22: 0R, Resistor_SMD:R_0603_1608Metric, F.Cu at (124.7, 62.5)
- C19, C20: footprint Capacitor_SMD:C_0603_1608Metric -> Capacitor_SMD:C_0402_1005Metric
- moved J10 62.9 mm to (177.3, 77.8)
- moved U4 40.6 mm to (195.8, 82.5)
- moved J7 37.5 mm to (186.9, 116.0), turned to 0 degrees
- moved J6 32.7 mm to (182.3, 116.0), turned to 0 degrees
- moved C20 31.3 mm to (154.5, 98.5), turned to -90 degrees
- moved C19 30.9 mm to (154.5, 96.6), turned to 90 degrees
- moved Y1 27.6 mm to (156.6, 97.1), turned to 0 degrees
- moved D1 27.5 mm to (125.5, 107.2)
- moved C37 27.1 mm to (140.4, 103.9), turned to -90 degrees
- moved J2 16.9 mm to (156.5, 92.3), turned to -90 degrees
- moved R19 14.9 mm to (158.0, 102.2)
- moved R18 14.1 mm to (156.5, 102.2)
- moved R17 13.2 mm to (155.0, 102.2)
- moved R16 12.2 mm to (153.5, 102.2)
- moved R4 7.57 mm to (140.0, 107.8)
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Connections:
- J10 pad 2: unconnected-(J10-Pin_2-Pad2) -> SDA
- J10 pad 3: unconnected-(J10-Pin_3-Pad3) -> SCL
- J10 pad 4: unconnected-(J10-Pin_4-Pad4) -> GND
- J2 pad 10: unconnected-(J2-~{RESET}-Pad10) -> RESET
- J2 pad 2: unconnected-(J2-SWDIO/TMS-Pad2) -> SWDIO
- J2 pad 3: Net-(J2-GND-Pad3) -> GND
- J2 pad 4: unconnected-(J2-SWCLK/TCK-Pad4) -> SWCLK
- J2 pad 5: Net-(J2-GND-Pad3) -> GND
- J2 pad 6: unconnected-(J2-SWO/TDO-Pad6) -> SWO
- J2 pad 9: unconnected-(J2-GNDDetect-Pad9) -> GND
- J9 pad 2: unconnected-(J9-Pin_2-Pad2) -> UART_TX
- J9 pad 3: unconnected-(J9-Pin_3-Pad3) -> UART_RX
- J9 pad 4: unconnected-(J9-Pin_4-Pad4) -> GND
- U1 pad 24: unconnected-(U1-SWCLK-Pad24) -> SWCLK
- U1 pad 25: unconnected-(U1-SWDIO-Pad25) -> SWDIO
- U1 pad 29: unconnected-(U1-GPIO18-Pad29) -> SWO
- U1 pad 30: unconnected-(U1-GPIO19-Pad30) -> RESET
- U1 pad 41: unconnected-(U1-GPIO29/ADC3-Pad41) -> TRIGGER
Routing:
- net LA_CH15: track 27.5 -> 11.5 mm
- net Net-(J3-Pin_19): track 2.43 -> 17.5 mm
- net LA_CH14: track 24.8 -> 9.87 mm
- net LA_CH13: track 22.0 -> 8.05 mm
- net Net-(J3-Pin_18): track 2.45 -> 16.0 mm
- net LA_CH12: track 19.2 -> 6.14 mm
- net Net-(J3-Pin_17): track 2.46 -> 14.5 mm
- net Net-(J3-Pin_16): track 2.47 -> 13.6 mm
- net SWDIO: track 0.00 -> 10.6 mm
- net SWCLK: track 0.00 -> 10.6 mm, vias 0 -> 2
- net Net-(U1-XIN): track 0.00 -> 10.4 mm
- net Net-(J3-Pin_4): track 2.47 -> 12.7 mm
- net Net-(U1-XOUT): track 0.00 -> 9.51 mm
- net SWO: track 0.00 -> 9.09 mm
- net Net-(J3-Pin_5): track 2.45 -> 10.9 mm
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
Commit message: v0.1
Parts:
- added C25: 100nF, Capacitor_SMD:C_0603_1608Metric, F.Cu at (138.5, 108.3)
- added C26: 100nF, Capacitor_SMD:C_0603_1608Metric, F.Cu at (210.0, 105.4)
- added C38: 100nF, Capacitor_SMD:C_0603_1608Metric, F.Cu at (210.0, 107.9)
- added C39: 100nF, Capacitor_SMD:C_0603_1608Metric, F.Cu at (149.4, 107.3)
- added J5: Conn_ARM_JTAG_SWD_10, Connector_PinHeader_1.27mm:PinHeader_2x05_P1.27mm_Vertical, F.Cu at (214.1, 103.3)
- added U6: SN74LVC8T245, Package_SO:TSSOP-24_4.4x7.8mm_P0.65mm, F.Cu at (144.1, 109.3)
- added U7: SN74LVC8T245, Package_SO:TSSOP-24_4.4x7.8mm_P0.65mm, F.Cu at (154.4, 109.3)
- R10, R11, R12, R13, R14, R15, R16, R17, R18, R19, R4, R5, R6, R7, R8, R9: moved to B.Cu
- moved C36 55.1 mm to (168.2, 106.0), turned to -90 degrees
- moved C29 46.9 mm to (95.8, 116.5)
- moved R19 38.9 mm to (131.5, 130.7)
- moved R18 36.9 mm to (133.0, 130.7)
- moved R17 35.0 mm to (134.5, 130.7)
- moved R15 34.1 mm to (127.9, 126.6)
- moved R16 33.4 mm to (136.0, 130.7)
- moved C35 32.6 mm to (145.1, 92.7), turned to 90 degrees
- moved C32 32.6 mm to (140.2, 93.5), turned to 180 degrees
- moved R14 31.6 mm to (129.4, 126.6)
- moved C31 29.9 mm to (138.5, 94.5), turned to 180 degrees
- moved R13 29.3 mm to (130.9, 126.6)
- moved R5 29.3 mm to (132.8, 135.7), turned to 90 degrees
- moved R8 29.3 mm to (137.2, 135.7), turned to 90 degrees
- moved R4 29.3 mm to (131.3, 135.7), turned to 90 degrees
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Connections:
- J3 pad 1: GND -> Net-(J3-Pin_1)
- J3 pad 18: Net-(J3-Pin_18) -> GND
- J3 pad 19: Net-(J3-Pin_19) -> GND
- J3 pad 20: Net-(J3-Pin_20) -> GND
- J3 pad 3: GND -> Net-(J3-Pin_3)
- R10 pad 2: Net-(J3-Pin_10) -> Net-(J3-Pin_7)
- R11 pad 2: Net-(J3-Pin_11) -> Net-(J3-Pin_8)
- R12 pad 2: Net-(J3-Pin_12) -> Net-(J3-Pin_9)
- R13 pad 2: Net-(J3-Pin_13) -> Net-(J3-Pin_10)
- R14 pad 2: Net-(J3-Pin_14) -> Net-(J3-Pin_11)
- R15 pad 2: Net-(J3-Pin_15) -> Net-(J3-Pin_12)
- R16 pad 2: Net-(J3-Pin_16) -> Net-(J3-Pin_13)
- R17 pad 2: Net-(J3-Pin_17) -> Net-(J3-Pin_14)
- R18 pad 2: Net-(J3-Pin_18) -> Net-(J3-Pin_15)
- R19 pad 2: Net-(J3-Pin_19) -> Net-(J3-Pin_16)
- R22 pad 1: VTREF -> VTREF_L
- R22 pad 2: Net-(J3-Pin_20) -> Net-(J3-Pin_17)
- R4 pad 2: Net-(J3-Pin_4) -> Net-(J3-Pin_1)
- R5 pad 2: Net-(J3-Pin_5) -> Net-(J3-Pin_2)
- R6 pad 2: Net-(J3-Pin_6) -> Net-(J3-Pin_3)
- R7 pad 2: Net-(J3-Pin_7) -> Net-(J3-Pin_4)
- R8 pad 2: Net-(J3-Pin_8) -> Net-(J3-Pin_5)
- R9 pad 2: Net-(J3-Pin_9) -> Net-(J3-Pin_6)
- U1 pad 1: Net-(U1-IOVDD-Pad1) -> 3V3
- U1 pad 10: Net-(U1-IOVDD-Pad1) -> 3V3
- U1 pad 11: LA_CH8 -> /LA_CH8_RP
- U1 pad 12: LA_CH9 -> /LA_CH9_RP
- U1 pad 13: LA_CH10 -> /LA_CH10_RP
- U1 pad 14: LA_CH11 -> /LA_CH11_RP
- U1 pad 15: LA_CH12 -> /LA_CH12_RP
- U1 pad 16: LA_CH13 -> /LA_CH13_RP
- U1 pad 17: LA_CH14 -> /LA_CH14_RP
- U1 pad 18: LA_CH15 -> /LA_CH15_RP
- U1 pad 2: LA_CH0 -> /LA_CH0_RP
- U1 pad 22: Net-(U1-IOVDD-Pad1) -> 3V3
- U1 pad 3: LA_CH1 -> /LA_CH1_RP
- U1 pad 33: Net-(U1-IOVDD-Pad1) -> 3V3
- U1 pad 4: LA_CH2 -> /LA_CH2_RP
- U1 pad 42: Net-(U1-IOVDD-Pad1) -> 3V3
- U1 pad 43: unconnected-(U1-ADC_AVDD-Pad43) -> 3V3
- U1 pad 44: unconnected-(U1-VREG_VIN-Pad44) -> 3V3
- U1 pad 48: unconnected-(U1-USB_VDD-Pad48) -> 3V3
- U1 pad 49: Net-(U1-IOVDD-Pad1) -> 3V3
- U1 pad 5: LA_CH3 -> /LA_CH3_RP
- U1 pad 6: LA_CH4 -> /LA_CH4_RP
- U1 pad 7: LA_CH5 -> /LA_CH5_RP
- U1 pad 8: LA_CH6 -> /LA_CH6_RP
- U1 pad 9: LA_CH7 -> /LA_CH7_RP
Routing:
- net Net-(J3-Pin_19): track 17.5 -> 0.00 mm
- net Net-(J3-Pin_18): track 16.0 -> 0.00 mm
- net Net-(J3-Pin_17): track 14.5 -> 0.00 mm
- net Net-(J3-Pin_16): track 13.6 -> 0.00 mm
- net /LA_CH15_RP: track 0.00 -> 12.9 mm
- net LA_CH11: track 12.8 -> 0.00 mm
- net Net-(J3-Pin_4): track 12.7 -> 0.00 mm
- net /LA_CH14_RP: track 0.00 -> 12.1 mm
- net LA_CH10: track 11.6 -> 0.00 mm
- net LA_CH15: track 11.5 -> 0.00 mm
- net /LA_CH13_RP: track 0.00 -> 11.4 mm
- net Net-(J3-Pin_5): track 10.9 -> 0.00 mm
- net /LA_CH11_RP: track 0.00 -> 10.7 mm
- net LA_CH9: track 10.6 -> 0.00 mm
- net /LA_CH10_RP: track 0.00 -> 10.6 mm
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Other:
- copper layers 2 -> 4

Commit message: v0
Parts:
- removed J6, J7: Conn_01x03_Socket, Connector_PinHeader_2.54mm:PinHeader_1x03_P2.54mm_Vertical
- removed R21: 47R, Resistor_SMD:R_0603_1608Metric
- R10, R11, R12, R13, R14, R15, R16, R17, R18, R19, R4, R5, R6, R7, R8, R9: moved to F.Cu
- moved C22 88.2 mm to (133.5, 108.1)
- moved C23 71.9 mm to (167.0, 92.7), turned to -90 degrees
- moved C38 70.9 mm to (139.2, 111.3), turned to 90 degrees
- moved C24 68.9 mm to (164.2, 97.8), turned to 180 degrees
- moved R22 65.8 mm to (160.3, 117.8), turned to -90 degrees
- moved C26 60.9 mm to (149.4, 111.3), turned to 90 degrees
- moved R20 38.8 mm to (157.7, 88.8), turned to 180 degrees
- moved U4 34.7 mm to (162.7, 93.1), turned to -90 degrees
- moved J10 34.3 mm to (143.3, 82.8)
- moved R19 27.5 mm to (155.8, 117.9)
- moved R18 24.5 mm to (153.9, 117.9)
- moved R15 21.9 mm to (148.0, 117.9)
- moved R17 21.6 mm to (151.9, 117.9)
- moved C36 19.9 mm to (150.0, 98.1), turned to 0 degrees
- moved R16 19.0 mm to (150.0, 117.9)
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Connections:
- C23 pad 1: unconnected-(C23-Pad1) -> VREF
- C23 pad 2: unconnected-(C23-Pad2) -> GND
- C24 pad 1: unconnected-(C24-Pad1) -> 3V3
- C24 pad 2: unconnected-(C24-Pad2) -> GND
- J10 pad 1: unconnected-(J10-Pin_1-Pad1) -> VREF
- J2 pad 1: unconnected-(J2-VTref-Pad1) -> VREF
- J4 pad 1: unconnected-(J4-Pin_1-Pad1) -> VREF
- J9 pad 1: unconnected-(J9-Pin_1-Pad1) -> VREF
- U4 pad 1: unconnected-(U4-A1-Pad1) -> CS
- U4 pad 19: unconnected-(U4-VCCB-Pad19) -> 3V3
- U4 pad 2: unconnected-(U4-VCCA-Pad2) -> VREF
- U4 pad 3: unconnected-(U4-A2-Pad3) -> SCK
- U4 pad 4: unconnected-(U4-A3-Pad4) -> MISO
- U4 pad 5: unconnected-(U4-A4-Pad5) -> MOSI
- U4 pad 6: unconnected-(U4-A5-Pad6) -> UART_RX
- U4 pad 7: unconnected-(U4-A6-Pad7) -> UART_TX
- U4 pad 8: unconnected-(U4-A7-Pad8) -> SDA
- U4 pad 9: unconnected-(U4-A8-Pad9) -> SCL
- U6 pad 10: unconnected-(U6-A8-Pad10) -> LA_CH7
- U6 pad 11: Net-(U6-GND-Pad11) -> GND
- U6 pad 12: Net-(U6-GND-Pad11) -> GND
- U6 pad 13: Net-(U6-GND-Pad11) -> GND
- U6 pad 3: unconnected-(U6-A1-Pad3) -> LA_CH0
- U6 pad 4: unconnected-(U6-A2-Pad4) -> LA_CH1
- U6 pad 5: unconnected-(U6-A3-Pad5) -> LA_CH2
- U6 pad 6: unconnected-(U6-A4-Pad6) -> LA_CH3
- U6 pad 7: unconnected-(U6-A5-Pad7) -> LA_CH4
- U6 pad 8: unconnected-(U6-A6-Pad8) -> LA_CH5
- U6 pad 9: unconnected-(U6-A7-Pad9) -> LA_CH6
- U7 pad 10: unconnected-(U7-A8-Pad10) -> LA_CH15
- U7 pad 11: Net-(U7-GND-Pad11) -> GND
- U7 pad 12: Net-(U7-GND-Pad11) -> GND
- U7 pad 13: Net-(U7-GND-Pad11) -> GND
- U7 pad 3: unconnected-(U7-A1-Pad3) -> LA_CH8
- U7 pad 4: unconnected-(U7-A2-Pad4) -> LA_CH9
- U7 pad 5: unconnected-(U7-A3-Pad5) -> LA_CH10
- U7 pad 6: unconnected-(U7-A4-Pad6) -> LA_CH11
- U7 pad 7: unconnected-(U7-A5-Pad7) -> LA_CH12
- U7 pad 8: unconnected-(U7-A6-Pad8) -> LA_CH13
- U7 pad 9: unconnected-(U7-A7-Pad9) -> LA_CH14
Routing:
- net 3V3: track 3.18 -> 35.9 mm, vias 0 -> 8
- net VTREF_L: track 0.00 -> 29.6 mm, vias 0 -> 3
- net SCL: track 0.00 -> 26.4 mm
- net SDA: track 0.00 -> 25.6 mm
- net /LS_OE: track 0.00 -> 24.3 mm
- net LA_CH0: track 0.00 -> 18.6 mm
- net UART_TX: track 0.00 -> 17.5 mm
- net LA_CH1: track 0.00 -> 17.1 mm
- net LA_CH2: track 0.00 -> 15.7 mm
- net UART_RX: track 0.00 -> 15.6 mm
- net LA_CH3: track 0.00 -> 14.3 mm
- net LA_CH4: track 0.00 -> 12.8 mm
- net LA_CH8: track 0.00 -> 12.4 mm
- net LA_CH5: track 0.00 -> 11.8 mm
- net LA_CH9: track 0.00 -> 11.5 mm
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Other:
- board size 52.7 x 29.1 mm -> 52.7 x 42.5 mm

Commit message: V0.11
Parts:
- added C40: 100nF, Capacitor_SMD:C_0603_1608Metric, F.Cu at (193.4, 75.7)
- added C41: 100nF, Capacitor_SMD:C_0603_1608Metric, F.Cu at (193.4, 78.2)
- added R21: 100k, Resistor_SMD:R_0603_1608Metric, F.Cu at (193.4, 80.7)
- added R23: 100k, Resistor_SMD:R_0603_1608Metric, F.Cu at (193.4, 83.2)
- added R24: 0R, Resistor_SMD:R_0603_1608Metric, F.Cu at (193.4, 85.7)
- added R25: 100k, Resistor_SMD:R_0603_1608Metric, F.Cu at (193.4, 88.2)
- added R26: 100k, Resistor_SMD:R_0603_1608Metric, F.Cu at (193.4, 90.7)
- added R27: 0R, Resistor_SMD:R_0603_1608Metric, F.Cu at (193.4, 93.2)
- moved J5 57.7 mm to (171.3, 97.7), turned to 180 degrees
- moved R20 13.1 mm to (162.4, 76.6)
- moved U4 3.08 mm to (163.7, 90.2)
- moved C23 3.07 mm to (168.0, 89.8)
- moved C24 3.07 mm to (165.2, 94.9)
- moved C33 2.07 mm to (136.6, 98.7)
- moved C35 0.98 mm to (145.8, 92.0), turned to 52 degrees
- moved C34 0.95 mm to (136.6, 99.7)
- moved J2 0.81 mm to (155.0, 93.1)
- moved C19 0.75 mm to (154.6, 97.4)
- moved C20 0.75 mm to (154.6, 99.2)
- moved Y1 0.75 mm to (156.7, 97.8)
Connections:
- net USB_M renamed USB_N
- J5 pad 10: unconnected-(J5-~{RESET}-Pad10) -> /TRESET
- J5 pad 2: unconnected-(J5-SWDIO/TMS-Pad2) -> /TSWDIO
- J5 pad 4: unconnected-(J5-SWCLK/TCK-Pad4) -> /TSWCLK
- U1 pad 27: unconnected-(U1-GPIO16-Pad27) -> /TSWDIO
- U1 pad 28: unconnected-(U1-GPIO17-Pad28) -> /TSWCLK
- U1 pad 29: SWO -> /TRESET
- U1 pad 31: unconnected-(U1-GPIO20-Pad31) -> /R_UART_P
- U1 pad 32: unconnected-(U1-GPIO21-Pad32) -> /R_UART_N
- U1 pad 34: unconnected-(U1-GPIO22-Pad34) -> /R_SDA
- U1 pad 35: unconnected-(U1-GPIO23-Pad35) -> /R_SCL
- U1 pad 36: unconnected-(U1-GPIO24-Pad36) -> /R_MOSI
- U1 pad 37: unconnected-(U1-GPIO25-Pad37) -> /R_MISO
- U1 pad 38: unconnected-(U1-GPIO26/ADC0-Pad38) -> /R_SCK
- U1 pad 39: unconnected-(U1-GPIO27/ADC1-Pad39) -> /R_CS
- U1 pad 40: /LS_OE -> unconnected-(U1-GPIO28/ADC2-Pad40)
- U1 pad 41: TRIGGER -> /LS_OE
- U4 pad 12: unconnected-(U4-B8-Pad12) -> /R_SDA
- U4 pad 13: unconnected-(U4-B7-Pad13) -> /R_SCL
- U4 pad 14: unconnected-(U4-B6-Pad14) -> /R_UART_N
- U4 pad 15: unconnected-(U4-B5-Pad15) -> /R_UART_P
- U4 pad 16: unconnected-(U4-B4-Pad16) -> /R_MOSI
- U4 pad 17: unconnected-(U4-B3-Pad17) -> /R_MISO
- U4 pad 18: unconnected-(U4-B2-Pad18) -> /R_SCK
- U4 pad 20: unconnected-(U4-B1-Pad20) -> /R_CS
- U4 pad 8: SDA -> SCL
- U4 pad 9: SCL -> SDA
Routing:
- net GND: track 0.00 -> 34.0 mm, vias 0 -> 30
- net /R_CS: track 0.00 -> 31.5 mm
- net /TRESET: track 0.00 -> 29.9 mm, vias 0 -> 2
- net /R_SCK: track 0.00 -> 29.4 mm
- net /R_MISO: track 0.00 -> 27.7 mm
- net /R_MOSI: track 0.00 -> 25.9 mm
- net /LS_OE: track 24.3 -> 0.00 mm
- net /R_UART_P: track 0.00 -> 23.9 mm
- net /R_UART_N: track 0.00 -> 23.9 mm
- net /R_SCL: track 0.00 -> 23.8 mm
- net /TSWCLK: track 0.00 -> 23.5 mm
- net /TSWDIO: track 0.00 -> 23.1 mm
- net /R_SDA: track 0.00 -> 22.1 mm
- net 3V3: track 35.9 -> 50.7 mm, vias 8 -> 14
- net USB_N: track 6.58 -> 17.3 mm
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- added copper zone on F.Cu, net 3V3
- added copper zone on In2.Cu, net 3V3
- added copper zone on In1.Cu, net GND
